File: hardware/fan-controller.sch (KiCad schematic (older format))
At the start: 11 parts, among them J1 Screw Terminal, J2 Screw Terminal, U1 L4931-5.0, U2 ATtiny13A-PU

Commit message: Added support for voltage-controlled fans.
Parts:
- removed M?: Fan_3pin, symbol Motor:Fan_3pin
- added D1: 1N4007, Diode_THT:D_DO-41_SOD81_P10.16mm_Horizontal, symbol Diode:1N4007
- added M2: 4-Pin PWM Fan, symbol Motor:Fan_4pin
- added M2: 3-Pin Fan, symbol Motor:Fan
- added Q?: PN2222A, Package_TO_SOT_THT:TO-92_Inline, symbol Transistor_BJT:PN2222A
Connections:
- net labels added: PWM
- wire segments 49 -> 60
Other:
- note added: "3-Pin Voltage-Controlled Fan"
- note added: "4-Pin PWM Fan"
- moved on the sheet: C1, C2, C3, C4, J1, J2, R1, RV1, U1, U2
